File: reflowControl/reflowControl.kicad_pcb (KiCad board)
At the start: 0 parts

Commit message: test
Parts:
- added C1: 1u, Capacitor_SMD:C_0603_1608Metric_Pad1.08x0.95mm_HandSolder, F.Cu at (187.9, 82.3)
- added C2: 1u, Capacitor_SMD:C_0603_1608Metric_Pad1.08x0.95mm_HandSolder, F.Cu at (187.9, 84.8)
- added C3: 22p, Capacitor_SMD:C_0805_2012Metric_Pad1.18x1.45mm_HandSolder, F.Cu at (184.5, 98.7)
- added C4: 22p, Capacitor_SMD:C_0805_2012Metric_Pad1.18x1.45mm_HandSolder, F.Cu at (184.5, 101.7)
- added J1: 10118194-0001LF, localparts:CONN_10118194-0001LF_AMP, F.Cu at (209.1, 80.0)
- added U1: MAX6675ISA+, localparts:21-0041B_8_MXM-M, F.Cu at (186.2, 89.3)
- added U2: ATmega644PA-A, Package_QFP:TQFP-44_10x10mm_P0.8mm, F.Cu at (178.5, 79.5)
- added U3: 4N35, Package_DIP:DIP-6_W7.62mm, F.Cu at (172.9, 88.8)
- added U4: MIC5317-3.3xM5, Package_TO_SOT_SMD:SOT-23-5, F.Cu at (193.0, 99.5)
- added U5: FT231XS, Package_SO:SSOP-20_3.9x8.7mm_P0.635mm, F.Cu at (194.4, 91.9)
- added U6: 4N35, Package_DIP:DIP-6_W7.62mm, F.Cu at (172.9, 98.0)
- added Y1: Crystal, localparts:21-0041B_8_MXM-M, F.Cu at (186.2, 94.6)
Other:
- board outline added: 7 x 3 mm
- copper layers 0 -> 2
